Commit message: Made separate policies for rough and stairs terrain

File: assets/urdf/v6biped_urdf_v4_aug29/v6biped_urdf_v4_squarefoot_aug29.urdf (robot description, URDF)
Before this commit: robot v6biped_urdf_v4_squarefoot, 19 links, 18 joints
Links:
- removed link link_04_L_knee_rocker_1
- removed link link_05_L_knee_link_1
- removed link link_13_R_knee_rocker_1
- removed link link_14_R_knee_link_1
Joints:
- removed joint joint_04_L_knee_rocker_RIGID
- removed joint joint_05_L_knee_link_RIGID
- removed joint joint_13_R_knee_rocker_RIGID
- removed joint joint_14_R_knee_link_PASSIVE
- joint joint_06_L_ankle_rocker_RIGID: origin xyz=-0.0302 -0.008226 -0.281 rpy=0 0 0 -> xyz=-0.0002 -0.014826 -0.000 rpy=0 0 0; parent link_03_L_hip_x_COLLISION_1 -> link_07_L_shank_link_main_1
- joint joint_07_L_shank_link_main: axis 0.0 1.0 0.0 -> 0 1 0
- joint joint_15_R_ankle_rocker_RIGID: origin xyz=-0.0302 0.008226 -0.281 rpy=0 0 0 -> xyz=0.0002 0.014226 0.003 rpy=0 0 0; parent link_12_R_hip_x_COLLISION_1 -> link_16_R_shank_link_main_1
- joint joint_16_R_shank_link_main: axis 0.0 -1.0 0.0 -> 0 -1 0
